Commit message: urdf updated with sensors and joints

File: urdf/rover.urdf (robot description, URDF)
Before this commit: robot rover, 3 links, 2 joints
Links:
- added link camera, mass 0.5; collision box size=0.1 0.5 0.2; visual box size=0.1 0.5 0.2
- added link lidar, mass 0.5; collision cylinder length=0.1 radius=0.1; visual cylinder length=0.1 radius=0.1
- added link wheel_back_left, mass 2; collision cylinder length=0.1 radius=0.15; visual cylinder length=0.1 radius=0.15
- added link wheel_back_right, mass 2; collision cylinder length=0.1 radius=0.15; visual cylinder length=0.1 radius=0.15
Joints:
- added joint camera_joint: type fixed, parent base_link, child camera, origin xyz=-0.35 0 0.15 rpy=0 0.0 3.14, axis 0.0 0.0 1.0
- added joint lidar_joint: type fixed, parent base_link, child lidar, origin xyz=-0.43 0 0.0 rpy=0 0.0 1.57, axis 0.0 0.0 1.0
- added joint wheel_back_left_joint: type continuous, parent base_link, child wheel_back_left, origin xyz=-0.25 -0.4 0.0 rpy=1.57 0.0 0.0, axis 0.0 0.0 1.0
- added joint wheel_back_right_joint: type continuous, parent base_link, child wheel_back_right, origin xyz=-0.25 0.4 0.0 rpy=1.57 0.0 0.0, axis 0.0 0.0 1.0
